File: board/Tiny-up5k.kicad_pcb (KiCad board)
At the start: 2 copper layers, 17.8 x 35.6 mm, 37 parts, among them J1 CONN_01X14, J2 CONN_01X14, J5 Prog, SW1 SW_Push, U1 ICE40UP5K-SG48ITR, U2 MIC5504-3.3YM5, U3 DSC6001CI2A-016.0000T, U4 MIC5504-1.2YM5, U5 SST25VF016B, U6 USB_OTG

Commit message: Also fix SMD pad that should get no solder
Parts:
- J5: footprint Connector_PinHeader_2.54mm:PinHeader_2x03_P2.54mm_Vertical_SMD -> board:PinHeader_2x03_P2.54mm_Vertical_SMD_NoSolder
Changed lines of the file:
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@@
     (0 F.Cu signal hide)
     (31 B.Cu signal hide)
-    (32 B.Adhes user)
+    (32 B.Adhes user hide)
     (33 F.Adhes user hide)
-    (34 B.Paste user hide)
+    (34 B.Paste user)
     (35 F.Paste user hide)
     (36 B.SilkS user hide)
@@
     (44 Edge.Cuts user hide)
     (45 Margin user hide)
-    (46 B.CrtYd user hide)
-    (47 F.CrtYd user)
+    (46 B.CrtYd user)
+    (47 F.CrtYd user hide)
     (48 B.Fab user hide)
     (49 F.Fab user)
   )
   (setup
-    (last_trace_width 0.25)
+    (last_trace_width 0.1)
     (user_trace_width 0.1)
     (user_trace_width 0.15)
@@
     )
   )
-  (module Connector_PinHeader_2.54mm:PinHeader_2x03_P2.54mm_Vertical_SMD (layer B.Cu)
+  (module Package_SON:WSON-8-1EP_6x5mm_P1.27mm_EP3.4x4mm (layer F.Cu)
+    (at 151.0665 125.5395 180)
+    (descr "WSON, 8 Pin (http://ww1.microchip.com/downloads/en/AppNotes/S72030.pdf), generated with kicad-footprint-generator ipc_dfn_qfn_generator.py")
+    (tags "WSON DFN_QFN")
+    (attr smd)
+    (fp_text reference U5 (at 0 -3.45 180) (layer F.SilkS)
+      (effects (font (size 1 1) (thickness 0.15)))
+    )
+    (fp_text value SST25VF016B (at -8.9535 0.0635 180) (layer F.Fab)
+      (effects (font (size 1 1) (thickness 0.15)))
+    )
+    (fp_line (start 0 -2.61) (end 3 -2.61) (layer F.SilkS) (width 0.12))
+    (fp_line (start -3 2.61) (end 3 2.61) (layer F.SilkS) (width 0.12))
+    (fp_line (start -2 -2.5) (end 3 -2.5) (layer F.Fab) (width 0.1))
+    (fp_line (start 3 -2.5) (end 3 2.5) (layer F.Fab) (width 0.1))
+    (fp_line (start 3 2.5) (end -3 2.5) (layer F.Fab) (width 0.1))
+    (fp_line (start -3 2.5) (end -3 -1.5) (layer F.Fab) (width 0.1))
+    (fp_line (start -3 -1.5) (end -2 -2.5) (layer F.Fab) (width 0.1))
+    (fp_line (start -3.3 -2.75) (end -3.3 2.75) (layer F.CrtYd) (width 0.05))
+    (fp_line (start -3.3 2.75) (end 3.3 2.75) (layer F.CrtYd) (width 0.05))
+    (fp_line (start 3.3 2.75) (end 3.3 -2.75) (layer F.CrtYd) (width 0.05))
+    (fp_line (start 3.3 -2.75) (end -3.3 -2.75) (layer F.CrtYd) (width 0.05))
+    (fp_text user %R (at 0 0 180) (layer F.Fab)
+      (effects (font (size 1 1) (thickness 0.15)))
+    )
+    (pad 9 smd roundrect (at 0 0 180) (size 3.4 4) (layers F.Cu F.Mask) (roundrect_rratio 0.073529)
+      (net 7 GND))
+    (pad "" smd roundrect (at -0.85 -1 180) (size 1.37 1.61) (layers F.Paste) (roundrect_rratio 0.182482))
+    (pad "" smd roundrect (at -0.85 1 180) (size 1.37 1.61) (layers F.Paste) (roundrect_rratio 0.182482))
+    (pad "" smd roundrect (at 0.85 -1 180) (size 1.37 1.61) (layers F.Paste) (roundrect_rratio 0.182482))
+    (pad "" smd roundrect (at 0.85 1 180) (size 1.37 1.61) (layers F.Paste) (roundrect_rratio 0.182482))
+    (pad 1 smd roundrect (at -2.6625 -1.905 180) (size 0.775 0.5) (layers F.Cu F.Paste F.Mask) (roundrect_rratio 0.25)
+      (net 6 SS))
+    (pad 2 smd roundrect (at -2.6625 -0.635 180) (size 0.775 0.5) (layers F.Cu F.Paste F.Mask) (roundrect_rratio 0.25)
+      (net 5 SDI))
+    (pad 3 smd roundrect (at -2.6625 0.635 180) (size 0.775 0.5) (layers F.Cu F.Paste F.Mask) (roundrect_rratio 0.25)
+      (net 43 "Net-(R10-Pad2)"))
+    (pad 4 smd roundrect (at -2.6625 1.905 180) (size 0.775 0.5) (layers F.Cu F.Paste F.Mask) (roundrect_rratio 0.25)
+      (net 7 GND))
+    (pad 5 smd roundrect (at 2.6625 1.905 180) (size 0.775 0.5) (layers F.Cu F.Paste F.Mask) (roundrect_rratio 0.25)
+      (net 8 SDO))
+    (pad 6 smd roundrect (at 2.6625 0.635 180) (size 0.775 0.5) (layers F.Cu F.Paste F.Mask) (roundrect_rratio 0.25)
+      (net 3 SCK))
+    (pad 7 smd roundrect (at 2.6625 -0.635 180) (size 0.775 0.5) (layers F.Cu F.Paste F.Mask) (roundrect_rratio 0.25)
+      (net 42 "Net-(R7-Pad2)"))
+    (pad 8 smd roundrect (at 2.6625 -1.905 180) (size 0.775 0.5) (layers F.Cu F.Paste F.Mask) (roundrect_rratio 0.25)
+      (net 15 SPI_VCCIO1))
+    (model ${KISYS3DMOD}/Package_SON.3dshapes/WSON-8-1EP_6x5mm_P1.27mm_EP3.4x4mm.wrl
+      (at (xyz 0 0 0))
+      (scale (xyz 1 1 1))
+      (rotate (xyz 0 0 0))
+    )
+  )
+  (module board:PinHeader_2x03_P2.54mm_Vertical_SMD_NoSolder (layer B.Cu)
     (at 151.145 128.905)
     (descr "surface-mounted straight pin header, 2x03, 2.54mm pitch, double rows")
     (tags "Surface mounted pin header SMD 2x03 2.54mm double row")
     (attr smd)
-    (fp_text reference J5 (at 0 -4.0005) (layer B.SilkS)
+    (fp_text reference J5 (at 0 4.87) (layer B.SilkS)
       (effects (font (size 1 1) (thickness 0.15)) (justify mirror))
     )
@@
       (effects (font (size 1 1) (thickness 0.15)) (justify mirror))
     )
-    (pad 1 smd rect (at -2.525 2.54) (size 3.15 1) (layers B.Cu B.Paste B.Mask)
-      (net 7 GND))
-    (pad 2 smd rect (at 2.525 2.54) (size 3.15 1) (layers B.Cu B.Paste B.Mask)
+    (pad 1 smd rect (at -2.525 2.54) (size 3.15 1) (layers B.Cu B.Mask)
+      (net 7 GND))
+    (pad 2 smd rect (at 2.525 2.54) (size 3.15 1) (layers B.Cu B.Mask)
       (net 3 SCK))
-    (pad 3 smd rect (at -2.525 0) (size 3.15 1) (layers B.Cu B.Paste B.Mask)
-      (net 15 SPI_VCCIO1))
-    (pad 4 smd rect (at 2.525 0) (size 3.15 1) (layers B.Cu B.Paste B.Mask)
+    (pad 3 smd rect (at -2.525 0) (size 3.15 1) (layers B.Cu B.Mask)
+      (net 15 SPI_VCCIO1))
+    (pad 4 smd rect (at 2.525 0) (size 3.15 1) (layers B.Cu B.Mask)
       (net 8 SDO))
-    (pad 5 smd rect (at -2.525 -2.54) (size 3.15 1) (layers B.Cu B.Paste B.Mask)
+    (pad 5 smd rect (at -2.525 -2.54) (size 3.15 1) (layers B.Cu B.Mask)
       (net 6 SS))
-    (pad 6 smd rect (at 2.525 -2.54) (size 3.15 1) (layers B.Cu B.Paste B.Mask)
+    (pad 6 smd rect (at 2.525 -2.54) (size 3.15 1) (layers B.Cu B.Mask)
       (net 5 SDI))
-  )
-  (module Package_SON:WSON-8-1EP_6x5mm_P1.27mm_EP3.4x4mm (layer F.Cu)
-    (at 151.0665 125.5395 180)
-    (descr "WSON, 8 Pin (http://ww1.microchip.com/downloads/en/AppNotes/S72030.pdf), generated with kicad-footprint-generator ipc_dfn_qfn_generator.py")
-    (tags "WSON DFN_QFN")
-    (attr smd)
-    (fp_text reference U5 (at 0 -3.45 180) (layer F.SilkS)
-      (effects (font (size 1 1) (thickness 0.15)))
-    )
-    (fp_text value SST25VF016B (at -8.9535 0.0635 180) (layer F.Fab)
-      (effects (font (size 1 1) (thickness 0.15)))
-    )
-    (fp_line (start 0 -2.61) (end 3 -2.61) (layer F.SilkS) (width 0.12))
-    (fp_line (start -3 2.61) (end 3 2.61) (layer F.SilkS) (width 0.12))
-    (fp_line (start -2 -2.5) (end 3 -2.5) (layer F.Fab) (width 0.1))
-    (fp_line (start 3 -2.5) (end 3 2.5) (layer F.Fab) (width 0.1))
-    (fp_line (start 3 2.5) (end -3 2.5) (layer F.Fab) (width 0.1))
-    (fp_line (start -3 2.5) (end -3 -1.5) (layer F.Fab) (width 0.1))
-    (fp_line (start -3 -1.5) (end -2 -2.5) (layer F.Fab) (width 0.1))
-    (fp_line (start -3.3 -2.75) (end -3.3 2.75) (layer F.CrtYd) (width 0.05))
-    (fp_line (start -3.3 2.75) (end 3.3 2.75) (layer F.CrtYd) (width 0.05))
-    (fp_line (start 3.3 2.75) (end 3.3 -2.75) (layer F.CrtYd) (width 0.05))
-    (fp_line (start 3.3 -2.75) (end -3.3 -2.75) (layer F.CrtYd) (width 0.05))
-    (fp_text user %R (at 0 0 180) (layer F.Fab)
-      (effects (font (size 1 1) (thickness 0.15)))
-    )
-    (pad 9 smd roundrect (at 0 0 180) (size 3.4 4) (layers F.Cu F.Mask) (roundrect_rratio 0.073529)
-      (net 7 GND))
-    (pad "" smd roundrect (at -0.85 -1 180) (size 1.37 1.61) (layers F.Paste) (roundrect_rratio 0.182482))
-    (pad "" smd roundrect (at -0.85 1 180) (size 1.37 1.61) (layers F.Paste) (roundrect_rratio 0.182482))
-    (pad "" smd roundrect (at 0.85 -1 180) (size 1.37 1.61) (layers F.Paste) (roundrect_rratio 0.182482))
-    (pad "" smd roundrect (at 0.85 1 180) (size 1.37 1.61) (layers F.Paste) (roundrect_rratio 0.182482))
-    (pad 1 smd roundrect (at -2.6625 -1.905 180) (size 0.775 0.5) (layers F.Cu F.Paste F.Mask) (roundrect_rratio 0.25)
-      (net 6 SS))
-    (pad 2 smd roundrect (at -2.6625 -0.635 180) (size 0.775 0.5) (layers F.Cu F.Paste F.Mask) (roundrect_rratio 0.25)
-      (net 5 SDI))
-    (pad 3 smd roundrect (at -2.6625 0.635 180) (size 0.775 0.5) (layers F.Cu F.Paste F.Mask) (roundrect_rratio 0.25)
-      (net 43 "Net-(R10-Pad2)"))
-    (pad 4 smd roundrect (at -2.6625 1.905 180) (size 0.775 0.5) (layers F.Cu F.Paste F.Mask) (roundrect_rratio 0.25)
-      (net 7 GND))
-    (pad 5 smd roundrect (at 2.6625 1.905 180) (size 0.775 0.5) (layers F.Cu F.Paste F.Mask) (roundrect_rratio 0.25)
-      (net 8 SDO))
-    (pad 6 smd roundrect (at 2.6625 0.635 180) (size 0.775 0.5) (layers F.Cu F.Paste F.Mask) (roundrect_rratio 0.25)
-      (net 3 SCK))
-    (pad 7 smd roundrect (at 2.6625 -0.635 180) (size 0.775 0.5) (layers F.Cu F.Paste F.Mask) (roundrect_rratio 0.25)
-      (net 42 "Net-(R7-Pad2)"))
-    (pad 8 smd roundrect (at 2.6625 -1.905 180) (size 0.775 0.5) (layers F.Cu F.Paste F.Mask) (roundrect_rratio 0.25)
-      (net 15 SPI_VCCIO1))
-    (model ${KISYS3DMOD}/Package_SON.3dshapes/WSON-8-1EP_6x5mm_P1.27mm_EP3.4x4mm.wrl
-      (at (xyz 0 0 0))
-      (scale (xyz 1 1 1))
+    (model ${KISYS3DMOD}/Connector_PinHeader_2.54mm.3dshapes/PinHeader_2x03_P2.54mm_Vertical_SMD.wrl
+      (at (xyz 0 0 0))
+      (scale (xyz 1 1 1))
